Commit message: AR3 UI started

File: src/ar3/urdf/AR3_Empty.xacro (robot description, xacro)
@@ -1,5 +1,5 @@
 <?xml version="1.0"?>
 <!-- Revolute-Revolute Manipulator -->
-<robot name="AR3_Pedestal" xmlns:xacro="http://www.ros.org/wiki/xacro">
+<robot name="AR3" xmlns:xacro="http://www.ros.org/wiki/xacro">
   <!-- Constants for robot dimensions -->
   <xacro:property name="PI" value="3.1415926535897931"/>
@@ -17,5 +17,5 @@
     <parent link="world"/>
     <child link="base"/>
-    <origin xyz="0 0 1" rpy="0 0 0"/>
+    <origin xyz="0 0 0.08763" rpy="0 0 0"/>
     <axis xyz="0 0 1"/>
     <dynamics damping="0.7"/>

File: src/ar3/urdf/AR3_noGazebo.xacro (robot description, xacro)
@@ -268,5 +268,5 @@
   <link name="flange"/>
   <!-- Flange joint -->
-  <joint name="flange_joint" type="continuous">
+  <joint name="flange_joint" type="fixed">
     <parent link="link6"/>
     <child link="flange"/>

File: src/sim_control/src/AR3_noGazebo.urdf (robot description, URDF)
Before this commit: robot ar3, 9 links, 8 joints
Joints:
- joint flange_joint: type continuous -> fixed
