Commit message: Gazebo model now uses updated URDF

File: src/ar3/urdf/AR3.xacro (robot description, xacro)
@@ -20,13 +20,13 @@
   <xacro:property name="joint3_y" value="0"/>
   <xacro:property name="joint3_z" value=".305"/>
-  <xacro:property name="joint4_x" value="-.038"/>
-  <xacro:property name="joint4_y" value="-.0503"/>
-  <xacro:property name="joint4_z" value="0"/>
+  <xacro:property name="joint4_x" value="-0.036"/>
+  <xacro:property name="joint4_y" value="0"/>
+  <xacro:property name="joint4_z" value="0.05"/>
   <xacro:property name="joint5_x" value="0"/>
-  <xacro:property name="joint5_y" value="-.172"/>
-  <xacro:property name="joint5_z" value="0"/>
+  <xacro:property name="joint5_y" value="0"/>
+  <xacro:property name="joint5_z" value="0.172"/>
   <xacro:property name="joint6_x" value="0"/>
-  <xacro:property name="joint6_y" value="-.0149"/>
-  <xacro:property name="joint6_z" value="0"/>
+  <xacro:property name="joint6_y" value="0"/>
+  <xacro:property name="joint6_z" value="0.015"/>
   <!-- Import all Gazebo-customization elements, including Gazebo colors -->
   <xacro:include filename="$(find ar3)/urdf/AR3.gazebo" />
@@ -61,7 +61,7 @@
   <!-- Robot to Environment-->
   <!-- <joint name="BaseJoint" type="fixed">
-    <parent link="stand"/>
+    <parent link="world"/>
     <child link="base"/>
-    <origin xyz="0 0 .25" rpy="0 0 0"/>
+    <origin xyz="0 0 0" rpy="0 0 0"/>
     <axis xyz="0 0 1"/>
     <dynamics damping="0.7"/>
@@ -162,5 +162,5 @@
     <parent link="link2"/>
     <child link="link3"/>
-    <origin xyz="${joint3_x} ${joint3_y} ${joint3_z}" rpy="${-PI/2} 0 0"/>
+    <origin xyz="${joint3_x} ${joint3_y} ${joint3_z}" rpy="0 0 0"/>
     <axis xyz="1 0 0"/>
     <dynamics damping="0.7"/>
@@ -196,5 +196,5 @@
     <child link="link4"/>
     <origin xyz="${joint4_x} ${joint4_y} ${joint4_z}" rpy="0 0 0"/>
-    <axis xyz="0 1 0"/>
+    <axis xyz="0 0 1"/>
     <dynamics damping="0.7"/>
     <limit lower="${-PI/2}" upper="${PI/2}" effort="30.0" velocity="10.0"/>
@@ -262,5 +262,5 @@
     <child link="link6"/>
     <origin xyz="${joint6_x} ${joint6_y} ${joint6_z}" rpy="0 0 0"/>
-    <axis xyz="0 1 0"/>
+    <axis xyz="0 0 1"/>
     <dynamics damping="0.7"/>
   </joint>

Commit message: Interpreters added to interface AR3 with Rviz

File: src/ar3/urdf/AR3.xacro (robot description, xacro)
@@ -31,8 +31,4 @@
   <!-- Import all Gazebo-customization elements, including Gazebo colors -->
   <xacro:include filename="$(find ar3)/urdf/AR3.gazebo" />
-  <!-- Import Rviz colors -->
-  <xacro:include filename="$(find ar3)/urdf/materials.xacro" />
-  <!-- Used for fixing robot to Gazebo 'base_link' -->
-  <!-- <link name="world"/> -->
   <!-- BASE -->
   <link name="base">
@@ -59,12 +55,4 @@
     </inertial>
   </link>
-  <!-- Robot to Environment-->
-  <!-- <joint name="BaseJoint" type="fixed">
-    <parent link="world"/>
-    <child link="base"/>
-    <origin xyz="0 0 0" rpy="0 0 0"/>
-    <axis xyz="0 0 1"/>
-    <dynamics damping="0.7"/>
-  </joint> -->
   <!-- Link 1 -->
   <link name="link1">
@@ -92,5 +80,5 @@
   </link>
   <!-- JOINT 1 -->
-  <joint name="joint1" type="continuous">
+  <joint name="joint1" type="revolute">
     <parent link="base"/>
     <child link="link1"/>
@@ -98,5 +86,5 @@
     <axis xyz="0 0 1"/>
     <dynamics damping="0.7"/>
-    <limit lower="${-PI/2}" upper="${PI/2}" effort="30.0" velocity="10.0"/>
+    <limit lower="-2.0" upper="2.0" effort="30.0" velocity="10.0"/>
   </joint>
   <!-- Link 2 -->
@@ -124,7 +112,6 @@
     </inertial>
   </link>
-  <!-- LEFT OFF HERE ON JOINT 2 Z -->
   <!-- JOINT 2 -->
-  <joint name="joint2" type="continuous">
+  <joint name="joint2" type="revolute">
     <parent link="link1"/>
     <child link="link2"/>
@@ -132,5 +119,5 @@
     <axis xyz="1 0 0"/>
     <dynamics damping="0.7"/>
-    <limit lower="${-PI/2}" upper="${PI}" effort="30.0" velocity="10.0"/>
+    <limit lower="-2.0" upper="2.0" effort="30.0" velocity="10.0"/>
   </joint>
   <!-- Link 3 -->
@@ -159,5 +146,5 @@
   </link>
   <!-- JOINT 3 -->
-  <joint name="joint3" type="continuous">
+  <joint name="joint3" type="revolute">
     <parent link="link2"/>
     <child link="link3"/>
@@ -165,5 +152,5 @@
     <axis xyz="1 0 0"/>
     <dynamics damping="0.7"/>
-    <limit lower="${-PI/2}" upper="${PI/2}" effort="30.0" velocity="10.0"/>
+    <limit lower="-2.0" upper="2.0" effort="30.0" velocity="10.0"/>
   </joint>
   <!-- LINK 4-->
@@ -180,5 +167,5 @@
 	      <mesh filename="$(find ar3)/urdf/meshes/Link4.stl" scale=".001 .001 .001"/>
       </geometry>
-      <material name="orange"/>
+      <material name="blue"/>
     </visual>
     <inertial>
@@ -192,5 +179,5 @@
   </link>
   <!-- JOINT 4 -->
-  <joint name="joint4" type="continuous">
+  <joint name="joint4" type="revolute">
     <parent link="link3"/>
     <child link="link4"/>
@@ -198,5 +185,5 @@
     <axis xyz="0 0 1"/>
     <dynamics damping="0.7"/>
-    <limit lower="${-PI/2}" upper="${PI/2}" effort="30.0" velocity="10.0"/>
+    <limit lower="-2.0" upper="2.0" effort="30.0" velocity="10.0"/>
   </joint>
   <!-- LINK 5-->
@@ -225,5 +212,5 @@
   </link>
   <!-- JOINT 5 -->
-  <joint name="joint5" type="continuous">
+  <joint name="joint5" type="revolute">
     <parent link="link4"/>
     <child link="link5"/>
@@ -231,5 +218,5 @@
     <axis xyz="1 0 0"/>
     <dynamics damping="0.7"/>
-    <limit lower="${-PI/2}" upper="${PI/2}" effort="30.0" velocity="10.0"/>
+    <limit lower="-2.0" upper="2.0" effort="30.0" velocity="10.0"/>
   </joint>
   <!-- LINK 6-->
@@ -246,5 +233,5 @@
 	      <mesh filename="$(find ar3)/urdf/meshes/Link6.stl" scale=".001 .001 .001"/>
       </geometry>
-      <material name="orange"/>
+      <material name="blue"/>
     </visual>
     <inertial>
@@ -258,5 +245,5 @@
   </link>
   <!-- JOINT 6 -->
-  <joint name="joint6" type="continuous">
+  <joint name="joint6" type="revolute">
     <parent link="link5"/>
     <child link="link6"/>
@@ -264,66 +251,6 @@
     <axis xyz="0 0 1"/>
     <dynamics damping="0.7"/>
-  </joint>
-  <!-- GAZEBO ROS CONTROL SPECIFIC INFORMATION -->
-  <transmission name="tran1">
-    <type>transmission_interface/SimpleTransmission</type>
-    <joint name="joint1">
-      <hardwareInterface>hardware_interface/EffortJointInterface</hardwareInterface>
-    </joint>
-    <actuator name="motor1">
-      <hardwareInterface>hardware_interface/EffortJointInterface</hardwareInterface>
-      <mechanicalReduction>1</mechanicalReduction>
-    </actuator>
-  </transmission>
-  <transmission name="tran2">
-    <type>transmission_interface/SimpleTransmission</type>
-    <joint name="joint2">
-      <hardwareInterface>hardware_interface/EffortJointInterface</hardwareInterface>
-    </joint>
-    <actuator name="motor2">
-      <hardwareInterface>hardware_interface/EffortJointInterface</hardwareInterface>
-      <mechanicalReduction>1</mechanicalReduction>
-    </actuator>
-  </transmission>
-  <transmission name="tran3">
-    <type>transmission_interface/SimpleTransmission</type>
-    <joint name="joint3">
-      <hardwareInterface>hardware_interface/EffortJointInterface</hardwareInterface>
-    </joint>
-    <actuator name="motor3">
-      <hardwareInterface>hardware_interface/EffortJointInterface</hardwareInterface>
-      <mechanicalReduction>1</mechanicalReduction>
-    </actuator>
-  </transmission>
-  <transmission name="tran4">
-    <type>transmission_interface/SimpleTransmission</type>
-    <joint name="joint4">
-      <hardwareInterface>hardware_interface/EffortJointInterface</hardwareInterface>
-    </joint>
-    <actuator name="motor4">
-      <hardwareInterface>hardware_interface/EffortJointInterface</hardwareInterface>
-      <mechanicalReduction>1</mechanicalReduction>
-    </actuator>
-  </transmission>
-  <transmission name="tran5">
-    <type>transmission_interface/SimpleTransmission</type>
-    <joint name="joint5">
-      <hardwareInterface>hardware_interface/EffortJointInterface</hardwareInterface>
-    </joint>
-    <actuator name="motor5">
-      <hardwareInterface>hardware_interface/EffortJointInterface</hardwareInterface>
-      <mechanicalReduction>1</mechanicalReduction>
-    </actuator>
-  </transmission>
-  <transmission name="tran6">
-    <type>transmission_interface/SimpleTransmission</type>
-    <joint name="joint6">
-      <hardwareInterface>hardware_interface/EffortJointInterface</hardwareInterface>
-    </joint>
-    <actuator name="motor6">
-      <hardwareInterface>hardware_interface/EffortJointInterface</hardwareInterface>
-      <mechanicalReduction>1</mechanicalReduction>
-    </actuator>
-  </transmission>
+    <limit lower="-2.0" upper="2.0" effort="30.0" velocity="10.0"/>
+  </joint>
 <!-- END OF ROBOT -->
 </robot>

File: src/ar3/urdf/AR3_Empty.xacro (robot description, xacro)
@@ -11,6 +11,69 @@
   <!-- Used for fixing robot to Gazebo 'base_link' -->
   <link name="world"/>
+  <!-- Import Rviz colors -->
+  <xacro:include filename="$(find ar3)/urdf/materials.xacro" />
   <!-- Import all Gazebo-customization elements, including Gazebo colors -->
   <xacro:include filename="$(find ar3)/urdf/AR3.xacro" />
+  <!-- GAZEBO ROS CONTROL SPECIFIC INFORMATION -->
+  <transmission name="tran1">
+    <type>transmission_interface/SimpleTransmission</type>
+    <joint name="joint1">
+      <hardwareInterface>hardware_interface/EffortJointInterface</hardwareInterface>
+    </joint>
+    <actuator name="motor1">
+      <hardwareInterface>hardware_interface/EffortJointInterface</hardwareInterface>
+      <mechanicalReduction>1</mechanicalReduction>
+    </actuator>
+  </transmission>
+  <transmission name="tran2">
+    <type>transmission_interface/SimpleTransmission</type>
+    <joint name="joint2">
+      <hardwareInterface>hardware_interface/EffortJointInterface</hardwareInterface>
+    </joint>
+    <actuator name="motor2">
+      <hardwareInterface>hardware_interface/EffortJointInterface</hardwareInterface>
+      <mechanicalReduction>1</mechanicalReduction>
+    </actuator>
+  </transmission>
+  <transmission name="tran3">
+    <type>transmission_interface/SimpleTransmission</type>
+    <joint name="joint3">
+      <hardwareInterface>hardware_interface/EffortJointInterface</hardwareInterface>
+    </joint>
+    <actuator name="motor3">
+      <hardwareInterface>hardware_interface/EffortJointInterface</hardwareInterface>
+      <mechanicalReduction>1</mechanicalReduction>
+    </actuator>
+  </transmission>
+  <transmission name="tran4">
+    <type>transmission_interface/SimpleTransmission</type>
+    <joint name="joint4">
+      <hardwareInterface>hardware_interface/EffortJointInterface</hardwareInterface>
+    </joint>
+    <actuator name="motor4">
+      <hardwareInterface>hardware_interface/EffortJointInterface</hardwareInterface>
+      <mechanicalReduction>1</mechanicalReduction>
+    </actuator>
+  </transmission>
+  <transmission name="tran5">
+    <type>transmission_interface/SimpleTransmission</type>
+    <joint name="joint5">
+      <hardwareInterface>hardware_interface/EffortJointInterface</hardwareInterface>
+    </joint>
+    <actuator name="motor5">
+      <hardwareInterface>hardware_interface/EffortJointInterface</hardwareInterface>
+      <mechanicalReduction>1</mechanicalReduction>
+    </actuator>
+  </transmission>
+  <transmission name="tran6">
+    <type>transmission_interface/SimpleTransmission</type>
+    <joint name="joint6">
+      <hardwareInterface>hardware_interface/EffortJointInterface</hardwareInterface>
+    </joint>
+    <actuator name="motor6">
+      <hardwareInterface>hardware_interface/EffortJointInterface</hardwareInterface>
+      <mechanicalReduction>1</mechanicalReduction>
+    </actuator>
+  </transmission>
   <!-- Robot to Environment-->
   <joint name="BaseJoint" type="fixed">

File: src/ar3/urdf/AR3_noGazebo.urdf (robot description, URDF)
Before this commit: robot ar3, 9 links, 8 joints
Joints:
- joint joint1: limit lower=-1.57079632679 upper=1.57079632679 effort=30.0 velocity=10.0 -> lower=-2.0 upper=2.0 effort=30.0 velocity=10.0; type continuous -> revolute
- joint joint2: limit lower=-1.57079632679 upper=3.14159265359 effort=30.0 velocity=10.0 -> lower=-2.0 upper=2.0 effort=30.0 velocity=10.0; type continuous -> revolute
- joint joint3: limit lower=-1.57079632679 upper=1.57079632679 effort=30.0 velocity=10.0 -> lower=-2.0 upper=2.0 effort=30.0 velocity=10.0; type continuous -> revolute
- joint joint4: limit lower=-1.57079632679 upper=1.57079632679 effort=30.0 velocity=10.0 -> lower=-2.0 upper=2.0 effort=30.0 velocity=10.0; type continuous -> revolute
- joint joint5: limit lower=-1.57079632679 upper=1.57079632679 effort=30.0 velocity=10.0 -> lower=-2.0 upper=2.0 effort=30.0 velocity=10.0; type continuous -> revolute
- joint joint6: limit (none) -> lower=-2.0 upper=2.0 effort=30.0 velocity=10.0; type continuous -> revolute

File: src/ar3/urdf/AR3_noGazebo.xacro (robot description, xacro)
@@ -36,28 +36,5 @@
   <!-- Used for fixing robot to Gazebo 'base_link' -->
   <link name="world"/>
-  <!-- BASE -->
-  <link name="base">
-    <collision>
-      <origin xyz="0 0 0" rpy="0 0 0"/>
-      <geometry>
-	      <mesh filename="$(find ar3)/urdf/meshes/Base.stl" scale=".001 .001 .001"/>
-      </geometry>
-    </collision>
-    <visual>
-      <origin xyz="0 0 0" rpy="0 0 0"/>
-      <geometry>
-	      <mesh filename="$(find ar3)/urdf/meshes/Base.stl" scale=".001 .001 .001"/>
-      </geometry>
-      <material name="orange"/>
-    </visual>
-    <inertial>
-      <origin xyz="0 0 0" rpy="0 0 0"/>
-      <mass value="${mass}"/>
-      <inertia
-	      ixx="${mass / 12.0 * (width*width + height1*height1)}" ixy="0.0" ixz="0.0"
-	      iyy="${mass / 12.0 * (height1*height1 + width*width)}" iyz="0.0"
-	      izz="${mass / 12.0 * (width*width + width*width)}"/>
-    </inertial>
-  </link>
+  <xacro:include filename="$(find ar3)/urdf/AR3.xacro" />
   <!-- Robot to Environment-->
   <joint name="BaseJoint" type="fixed">
@@ -65,202 +42,4 @@
     <child link="base"/>
     <origin xyz="0 0 0" rpy="0 0 0"/>
-    <axis xyz="0 0 1"/>
-    <dynamics damping="0.7"/>
-  </joint>
-  <!-- Link 1 -->
-  <link name="link1">
-    <collision>
-      <origin xyz="0 0 0" rpy="0 0 0"/>
-      <geometry>
-	      <mesh filename="$(find ar3)/urdf/meshes/Link1.stl" scale=".001 .001 .001"/>
-      </geometry>
-    </collision>
-    <visual>
-      <origin xyz="0 0 0" rpy="0 0 0"/>
-      <geometry>
-	      <mesh filename="$(find ar3)/urdf/meshes/Link1.stl" scale=".001 .001 .001"/>
-      </geometry>
-      <material name="orange"/>
-    </visual>
-    <inertial>
-      <origin xyz="0 0 0" rpy="0 0 0"/>
-      <mass value="${mass}"/>
-      <inertia
-	      ixx="${mass / 12.0 * (width*width + height1*height1)}" ixy="0.0" ixz="0.0"
-	      iyy="${mass / 12.0 * (height1*height1 + width*width)}" iyz="0.0"
-	      izz="${mass / 12.0 * (width*width + width*width)}"/>
-    </inertial>
-  </link>
-  <!-- JOINT 1 -->
-  <joint name="joint1" type="continuous">
-    <parent link="base"/>
-    <child link="link1"/>
-    <origin xyz="${joint1_x} ${joint1_y} ${joint1_z}" rpy="0 0 0"/>
-    <axis xyz="0 0 1"/>
-    <dynamics damping="0.7"/>
-    <limit lower="${-PI/2}" upper="${PI/2}" effort="30.0" velocity="10.0"/>
-  </joint>
-  <!-- Link 2 -->
-  <link name="link2">
-    <collision>
-      <origin xyz="0 0 0" rpy="0 0 0"/>
-      <geometry>
-	      <mesh filename="$(find ar3)/urdf/meshes/Link2.stl" scale=".001 .001 .001"/>
-      </geometry>
-    </collision>
-    <visual>
-      <origin xyz="0 0 0" rpy="0 0 0"/>
-      <geometry>
-	      <mesh filename="$(find ar3)/urdf/meshes/Link2.stl" scale=".001 .001 .001"/>
-      </geometry>
-      <material name="blue"/>
-    </visual>
-    <inertial>
-      <origin xyz="0 0 0" rpy="0 0 0"/>
-      <mass value="${mass}"/>
-      <inertia
-	      ixx="${mass / 3.0 * (width*width + height2*height2)}" ixy="0.0" ixz="0.0"
-	      iyy="${mass / 3.0 * (height2*height2 + width*width)}" iyz="0.0"
-	      izz="${mass / 3.0 * (width*width + width*width)}"/>
-    </inertial>
-  </link>
-  <!-- LEFT OFF HERE ON JOINT 2 Z -->
-  <!-- JOINT 2 -->
-  <joint name="joint2" type="continuous">
-    <parent link="link1"/>
-    <child link="link2"/>
-    <origin xyz="${joint2_x} ${joint2_y} ${joint2_z}" rpy="0 0 0"/>
-    <axis xyz="1 0 0"/>
-    <dynamics damping="0.7"/>
-    <limit lower="${-PI/2}" upper="${PI}" effort="30.0" velocity="10.0"/>
-  </joint>
-  <!-- Link 3 -->
-  <link name="link3">
-    <collision>
-      <origin xyz="0 0 0" rpy="0 0 0"/>
-      <geometry>
-	      <mesh filename="$(find ar3)/urdf/meshes/Link3.stl" scale=".001 .001 .001"/>
-      </geometry>
-    </collision>
-    <visual>
-      <origin xyz="0 0 0" rpy="0 0 0"/>
-      <geometry>
-	      <mesh filename="$(find ar3)/urdf/meshes/Link3.stl" scale=".001 .001 .001"/>
-      </geometry>
-      <material name="orange"/>
-    </visual>
-    <inertial>
-      <origin xyz="0 0 0" rpy="0 0 0"/>
-      <mass value="${mass}"/>
-      <inertia
-	      ixx="${mass / 3.0 * (width*width + height3*height3)}" ixy="0.0" ixz="0.0"
-	      iyy="${mass / 3.0 * (height3*height3 + width*width)}" iyz="0.0"
-	      izz="${mass / 3.0 * (width*width + width*width)}"/>
-    </inertial>
-  </link>
-  <!-- JOINT 3 -->
-  <joint name="joint3" type="continuous">
-    <parent link="link2"/>
-    <child link="link3"/>
-    <origin xyz="${joint3_x} ${joint3_y} ${joint3_z}" rpy="0 0 0"/>
-    <axis xyz="1 0 0"/>
-    <dynamics damping="0.7"/>
-    <limit lower="${-PI/2}" upper="${PI/2}" effort="30.0" velocity="10.0"/>
-  </joint>
-  <!-- LINK 4-->
-  <link name="link4">
-    <collision>
-      <origin xyz="0 0 0" rpy="0 0 0"/>
-      <geometry>
-	      <mesh filename="$(find ar3)/urdf/meshes/Link4.stl" scale=".001 .001 .001"/>
-      </geometry>
-    </collision>
-    <visual>
-      <origin xyz="0 0 0" rpy="0 0 0"/>
-      <geometry>
-	      <mesh filename="$(find ar3)/urdf/meshes/Link4.stl" scale=".001 .001 .001"/>
-      </geometry>
-      <material name="orange"/>
-    </visual>
-    <inertial>
-      <origin xyz="0 0 0" rpy="0 0 0"/>
-      <mass value="${mass}"/>
-      <inertia
-	      ixx="${mass / 12.0 * (width*width + height4*height4)}" ixy="0.0" ixz="0.0"
-	      iyy="${mass / 12.0 * (height4*height4 + width*width)}" iyz="0.0"
-	      izz="${mass / 12.0 * (width*width + width*width)}"/>
-    </inertial>
-  </link>
-  <!-- JOINT 4 -->
-  <joint name="joint4" type="continuous">
-    <parent link="link3"/>
-    <child link="link4"/>
-    <origin xyz="${joint4_x} ${joint4_y} ${joint4_z}" rpy="0 0 0"/>
-    <axis xyz="0 0 1"/>
-    <dynamics damping="0.7"/>
-    <limit lower="${-PI/2}" upper="${PI/2}" effort="30.0" velocity="10.0"/>
-  </joint>
-  <!-- LINK 5-->
-  <link name="link5">
-    <collision>
-      <origin xyz="0 0 0" rpy="0 0 0"/>
-      <geometry>
-	      <mesh filename="$(find ar3)/urdf/meshes/Link5.stl" scale=".001 .001 .001"/>
-      </geometry>
-    </collision>
-    <visual>
-      <origin xyz="0 0 0" rpy="0 0 0"/>
-      <geometry>
-	      <mesh filename="$(find ar3)/urdf/meshes/Link5.stl" scale=".001 .001 .001"/>
-      </geometry>
-      <material name="orange"/>
-    </visual>
-    <inertial>
-      <origin xyz="0 0 0" rpy="0 0 0"/>
-      <mass value="${mass}"/>
-      <inertia
-	      ixx="${mass / 12.0 * (width*width + height4*height4)}" ixy="0.0" ixz="0.0"
-	      iyy="${mass / 12.0 * (height4*height4 + width*width)}" iyz="0.0"
-	      izz="${mass / 12.0 * (width*width + width*width)}"/>
-    </inertial>
-  </link>
-  <!-- JOINT 5 -->
-  <joint name="joint5" type="continuous">
-    <parent link="link4"/>
-    <child link="link5"/>
-    <origin xyz="${joint5_x} ${joint5_y} ${joint5_z}" rpy="0 0 0"/>
-    <axis xyz="1 0 0"/>
-    <dynamics damping="0.7"/>
-    <limit lower="${-PI/2}" upper="${PI/2}" effort="30.0" velocity="10.0"/>
-  </joint>
-  <!-- LINK 6-->
-  <link name="link6">
-    <collision>
-      <origin xyz="0 0 0" rpy="0 0 0"/>
-      <geometry>
-	      <mesh filename="$(find ar3)/urdf/meshes/Link6.stl" scale=".001 .001 .001"/>
-      </geometry>
-    </collision>
-    <visual>
-      <origin xyz="0 0 0" rpy="0 0 0"/>
-      <geometry>
-	      <mesh filename="$(find ar3)/urdf/meshes/Link6.stl" scale=".001 .001 .001"/>
-      </geometry>
-      <material name="orange"/>
-    </visual>
-    <inertial>
-      <origin xyz="0 0 0" rpy="0 0 0"/>
-      <mass value="${mass}"/>
-      <inertia
-	      ixx="${mass / 12.0 * (width*width + height4*height4)}" ixy="0.0" ixz="0.0"
-	      iyy="${mass / 12.0 * (height4*height4 + width*width)}" iyz="0.0"
-	      izz="${mass / 12.0 * (width*width + width*width)}"/>
-    </inertial>
-  </link>
-  <!-- JOINT 6 -->
-  <joint name="joint6" type="continuous">
-    <parent link="link5"/>
-    <child link="link6"/>
-    <origin xyz="${joint6_x} ${joint6_y} ${joint6_z}" rpy="0 0 0"/>
     <axis xyz="0 0 1"/>
     <dynamics damping="0.7"/>

Commit message: Fixed URDF colors

File: src/ar3/urdf/AR3.xacro (robot description, xacro)
@@ -44,5 +44,5 @@
 	      <mesh filename="$(find ar3)/urdf/meshes/Base.stl" scale=".001 .001 .001"/>
       </geometry>
-      <material name="orange"/>
+      <material name="blue"/>
     </visual>
     <inertial>
