Commit message: Corrected URDF rotations and added Rviz support

File: src/ar3/urdf/AR3_noGazebo.urdf (robot description, URDF)
Before this commit: robot ar3, 9 links, 8 joints
Links:
- link base: geometry collision mesh filename=file:///home/kurt/Robotics/src/ar3/urdf/meshes/Base.stl scale=.001 .001 .001; visual mesh filename=file:///home/kurt/Robotics/src/ar3/urdf/meshes/Base.stl scale=.001 .001 .001
- link link1: geometry collision mesh filename=file:///home/kurt/Robotics/src/ar3/urdf/meshes/Link1.stl scale=.001 .001 .001; visual mesh filename=file:///home/kurt/Robotics/src/ar3/urdf/meshes/Link1.stl scale=.001 .001 .001
- link link2: geometry collision mesh filename=file:///home/kurt/Robotics/src/ar3/urdf/meshes/Link2.stl scale=.001 .001 .001; visual mesh filename=file:///home/kurt/Robotics/src/ar3/urdf/meshes/Link2.stl scale=.001 .001 .001
- link link3: geometry collision mesh filename=file:///home/kurt/Robotics/src/ar3/urdf/meshes/Link3.stl scale=.001 .001 .001; visual mesh filename=file:///home/kurt/Robotics/src/ar3/urdf/meshes/Link3.stl scale=.001 .001 .001
- link link4: geometry collision mesh filename=file:///home/kurt/Robotics/src/ar3/urdf/meshes/Link4.stl scale=.001 .001 .001; visual mesh filename=file:///home/kurt/Robotics/src/ar3/urdf/meshes/Link4.stl scale=.001 .001 .001
- link link5: geometry collision mesh filename=file:///home/kurt/Robotics/src/ar3/urdf/meshes/Link5.stl scale=.001 .001 .001; visual mesh filename=file:///home/kurt/Robotics/src/ar3/urdf/meshes/Link5.stl scale=.001 .001 .001
- link link6: geometry collision mesh filename=file:///home/kurt/Robotics/src/ar3/urdf/meshes/Link6.stl scale=.001 .001 .001; visual mesh filename=file:///home/kurt/Robotics/src/ar3/urdf/meshes/Link6.stl scale=.001 .001 .001
Joints:
- joint flange_joint: axis 0 1 0 -> 0 0 1; origin xyz=0 0 0 rpy=0 0 0 -> xyz=-0.003 0.020066 0.078 rpy=0 0 0; type continuous -> fixed
- joint joint3: origin xyz=-0.015 0 0.305 rpy=-1.57079632679 0 0 -> xyz=-0.015 0 0.305 rpy=0 0 0
- joint joint4: axis 0 1 0 -> 0 0 1; origin xyz=-0.038 -0.0503 0 rpy=0 0 0 -> xyz=-0.036 0 0.05 rpy=0 0 0
- joint joint5: origin xyz=0 -0.172 0 rpy=0 0 0 -> xyz=0 0 0.172 rpy=0 0 0
- joint joint6: axis 0 1 0 -> 0 0 1; origin xyz=0 -0.0149 0 rpy=0 0 0 -> xyz=0 0 0.015 rpy=0 0 0

File: src/ar3/urdf/AR3_noGazebo.xacro (robot description, xacro)
@@ -20,15 +20,16 @@
   <xacro:property name="joint3_y" value="0"/>
   <xacro:property name="joint3_z" value=".305"/>
-  <xacro:property name="joint4_x" value="-.038"/>
-  <xacro:property name="joint4_y" value="-.0503"/>
-  <xacro:property name="joint4_z" value="0"/>
+  <xacro:property name="joint4_x" value="-0.036"/>
+  <xacro:property name="joint4_y" value="0"/>
+  <xacro:property name="joint4_z" value="0.05"/>
   <xacro:property name="joint5_x" value="0"/>
-  <xacro:property name="joint5_y" value="-.172"/>
-  <xacro:property name="joint5_z" value="0"/>
+  <xacro:property name="joint5_y" value="0"/>
+  <xacro:property name="joint5_z" value="0.172"/>
   <xacro:property name="joint6_x" value="0"/>
-  <xacro:property name="joint6_y" value="-.0149"/>
-  <xacro:property name="joint6_z" value="0"/>
-  <!-- Import all Gazebo-customization elements, including Gazebo colors -->
-  <xacro:include filename="$(find ar3)/urdf/AR3.gazebo" />
+  <xacro:property name="joint6_y" value="0"/>
+  <xacro:property name="joint6_z" value="0.015"/>
+  <xacro:property name="tcp_x" value="-0.003"/>
+  <xacro:property name="tcp_y" value="0.020066"/>
+  <xacro:property name="tcp_z" value="0.078"/>
   <!-- Import Rviz colors -->
   <xacro:include filename="$(find ar3)/urdf/materials.xacro" />
@@ -162,5 +163,5 @@
     <parent link="link2"/>
     <child link="link3"/>
-    <origin xyz="${joint3_x} ${joint3_y} ${joint3_z}" rpy="${-PI/2} 0 0"/>
+    <origin xyz="${joint3_x} ${joint3_y} ${joint3_z}" rpy="0 0 0"/>
     <axis xyz="1 0 0"/>
     <dynamics damping="0.7"/>
@@ -196,5 +197,5 @@
     <child link="link4"/>
     <origin xyz="${joint4_x} ${joint4_y} ${joint4_z}" rpy="0 0 0"/>
-    <axis xyz="0 1 0"/>
+    <axis xyz="0 0 1"/>
     <dynamics damping="0.7"/>
     <limit lower="${-PI/2}" upper="${PI/2}" effort="30.0" velocity="10.0"/>
@@ -262,5 +263,5 @@
     <child link="link6"/>
     <origin xyz="${joint6_x} ${joint6_y} ${joint6_z}" rpy="0 0 0"/>
-    <axis xyz="0 1 0"/>
+    <axis xyz="0 0 1"/>
     <dynamics damping="0.7"/>
   </joint>
@@ -271,6 +272,6 @@
     <parent link="link6"/>
     <child link="flange"/>
-    <origin xyz="0 0 0" rpy="0 0 0"/>
-    <axis xyz="0 1 0"/>
+    <origin xyz="${tcp_x} ${tcp_y} ${tcp_z}" rpy="0 0 0"/>
+    <axis xyz="0 0 1"/>
     <dynamics damping="0.7"/>
   </joint>

Commit message: Runs on WSL now

File: src/ar3/urdf/AR3_noGazebo.urdf (robot description, URDF)
Before this commit: robot ar3, 9 links, 8 joints
Links:
- link base: geometry collision mesh filename=file:///home/kpdudek/Robotics/src/ar3/urdf/meshes/Base.stl scale=.001 .001 .001; visual mesh filename=file:///home/kpdudek/Robotics/src/ar3/urdf/meshes/Base.stl scale=.001 .001 .001
- link link1: geometry collision mesh filename=file:///home/kpdudek/Robotics/src/ar3/urdf/meshes/Link1.stl scale=.001 .001 .001; visual mesh filename=file:///home/kpdudek/Robotics/src/ar3/urdf/meshes/Link1.stl scale=.001 .001 .001
- link link2: geometry collision mesh filename=file:///home/kpdudek/Robotics/src/ar3/urdf/meshes/Link2.stl scale=.001 .001 .001; visual mesh filename=file:///home/kpdudek/Robotics/src/ar3/urdf/meshes/Link2.stl scale=.001 .001 .001
- link link3: geometry collision mesh filename=file:///home/kpdudek/Robotics/src/ar3/urdf/meshes/Link3.stl scale=.001 .001 .001; visual mesh filename=file:///home/kpdudek/Robotics/src/ar3/urdf/meshes/Link3.stl scale=.001 .001 .001
- link link4: geometry collision mesh filename=file:///home/kpdudek/Robotics/src/ar3/urdf/meshes/Link4.stl scale=.001 .001 .001; visual mesh filename=file:///home/kpdudek/Robotics/src/ar3/urdf/meshes/Link4.stl scale=.001 .001 .001
- link link5: geometry collision mesh filename=file:///home/kpdudek/Robotics/src/ar3/urdf/meshes/Link5.stl scale=.001 .001 .001; visual mesh filename=file:///home/kpdudek/Robotics/src/ar3/urdf/meshes/Link5.stl scale=.001 .001 .001
- link link6: geometry collision mesh filename=file:///home/kpdudek/Robotics/src/ar3/urdf/meshes/Link6.stl scale=.001 .001 .001; visual mesh filename=file:///home/kpdudek/Robotics/src/ar3/urdf/meshes/Link6.stl scale=.001 .001 .001

Commit message: GCode generator added

File: src/ar3/urdf/AR3_noGazebo.urdf (robot description, URDF)
Before this commit: robot ar3, 9 links, 8 joints
Joints:
- joint joint1: limit lower=-2.0 upper=2.0 effort=30.0 velocity=10.0 -> lower=-1.57 upper=1.57 effort=30.0 velocity=10.0
- joint joint2: limit lower=-2.0 upper=2.0 effort=30.0 velocity=10.0 -> lower=-0.5 upper=1.57 effort=30.0 velocity=10.0
- joint joint3: limit lower=-2.0 upper=2.0 effort=30.0 velocity=10.0 -> lower=-0.1 upper=2.0 effort=30.0 velocity=10.0
- joint joint4: limit lower=-2.0 upper=2.0 effort=30.0 velocity=10.0 -> lower=-1.57 upper=1.57 effort=30.0 velocity=10.0
- joint joint5: limit lower=-2.0 upper=2.0 effort=30.0 velocity=10.0 -> lower=-1.4 upper=1.4 effort=30.0 velocity=10.0
- joint joint6: limit lower=-2.0 upper=2.0 effort=30.0 velocity=10.0 -> lower=-3.14 upper=3.14 effort=30.0 velocity=10.0
