Commit message: UI Icons in repo now used

File: src/ar3/urdf/ar3.urdf (robot description, URDF)
Before this commit: robot ar3, 11 links, 10 joints
Links:
- link base: geometry collision mesh filename=file:///home/kurt/Robotics/src/ar3/urdf/meshes/Base.dae; visual mesh filename=file:///home/kurt/Robotics/src/ar3/urdf/meshes/Base.dae
- link eoat: geometry collision mesh filename=file:///home/kurt/Robotics/src/ar3/urdf/meshes/gripper.dae; visual mesh filename=file:///home/kurt/Robotics/src/ar3/urdf/meshes/gripper.dae
- link link1: geometry collision mesh filename=file:///home/kurt/Robotics/src/ar3/urdf/meshes/Link1.dae; visual mesh filename=file:///home/kurt/Robotics/src/ar3/urdf/meshes/Link1.dae
- link link2: geometry collision mesh filename=file:///home/kurt/Robotics/src/ar3/urdf/meshes/Link2.dae; visual mesh filename=file:///home/kurt/Robotics/src/ar3/urdf/meshes/Link2.dae
- link link3: geometry collision mesh filename=file:///home/kurt/Robotics/src/ar3/urdf/meshes/Link3.dae; visual mesh filename=file:///home/kurt/Robotics/src/ar3/urdf/meshes/Link3.dae
- link link4: geometry collision mesh filename=file:///home/kurt/Robotics/src/ar3/urdf/meshes/Link4.dae; visual mesh filename=file:///home/kurt/Robotics/src/ar3/urdf/meshes/Link4.dae
- link link5: geometry collision mesh filename=file:///home/kurt/Robotics/src/ar3/urdf/meshes/Link5.dae; visual mesh filename=file:///home/kurt/Robotics/src/ar3/urdf/meshes/Link5.dae
- link link6: geometry collision mesh filename=file:///home/kurt/Robotics/src/ar3/urdf/meshes/Link6.dae; visual mesh filename=file:///home/kurt/Robotics/src/ar3/urdf/meshes/Link6.dae
